File: mipt.kicad_sch (KiCad schematic)
At the start: 0 parts

Commit message: home work 3
Other:
- sheet home work 2 renamed Домашняя работа 2
- sheet home work 3 renamed Домашняя работа 3
Changed lines of the file:
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@@
 			(color 0 0 0 0.0000)
 		)
-		(property "Sheetname" "home work 2"
+		(property "Sheetname" "Домашняя работа 2"
 			(at 17.78 18.3384 0)
 			(effects
@@
 			(color 0 0 0 0.0000)
 		)
-		(property "Sheetname" "home work 3"
+		(property "Sheetname" "Домашняя работа 3"
 			(at 17.78 31.0384 0)
 			(effects

Commit message: home works 3 and 4
Other:
- added sheet Домашняя работа 4 (./home works/home work 04.kicad_sch)
Changed lines of the file:
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@@
+		)
+	)
+	(sheet
+		(at 17.78 44.45)
+		(size 34.29 6.35)
+		(fields_autoplaced yes)
+		(stroke
+			(width 0.1524)
+			(type solid)
+		)
+		(fill
+			(color 0 0 0 0.0000)
+		)
+		(property "Sheetname" "Домашняя работа 4"
+			(at 17.78 43.7384 0)
+			(effects
+				(font
+					(size 1.27 1.27)
+				)
+				(justify left bottom)
+			)
+		)
+		(property "Sheetfile" "./home works/home work 04.kicad_sch"
+			(at 17.78 51.3846 0)
+			(effects
+				(font
+					(size 1.27 1.27)
+				)
+				(justify left top)
+			)
+		)
+		(instances
+			(project "mipt"
+				(path "/34d483ea-61c1-4e08-b30a-5dee616d4777"
+					(page "7")
+				)
+			)
 		)
 	)
