File: mipt.kicad_sch (KiCad schematic)
At the start: 0 parts

Commit message: some fixes and add hw 5
Other:
- added sheet Домашняя работа 5 (./.home_works/home work 05.kicad_sch)
Changed lines of the file:
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@@
 	(paper "A4")
+	(sheet
+		(at 17.78 57.15)
+		(size 34.29 6.35)
+		(fields_autoplaced yes)
+		(stroke
+			(width 0.1524)
+			(type solid)
+		)
+		(fill
+			(color 0 0 0 0.0000)
+		)
+		(property "Sheetname" "Домашняя работа 5"
+			(at 17.78 56.4384 0)
+			(effects
+				(font
+					(size 1.27 1.27)
+				)
+				(justify left bottom)
+			)
+		)
+		(property "Sheetfile" "./.home_works/home work 05.kicad_sch"
+			(at 17.78 64.0846 0)
+			(effects
+				(font
+					(size 1.27 1.27)
+				)
+				(justify left top)
+			)
+		)
+		(instances
+			(project "mipt"
+				(path "/34d483ea-61c1-4e08-b30a-5dee616d4777"
+					(page "9")
+				)
+			)
+		)
+	)
 	(sheet
 		(at 17.78 19.05)
