File: home works/home work 03/task 02.kicad_sch (KiCad schematic)
At the start: 0 parts

Commit message: home work 3
Parts:
- added R11, R15: 220, symbol Device:R
- added R12: 430, symbol Device:R
- added R13, R17: 82, symbol Device:R
- added R14: ?, symbol Device:R
- added R16: 680, symbol Device:R
- added R18: 100, symbol Device:R
- added R19, R20: нагрузка 0.07A, symbol Device:R
Connections:
- new net +12V7: R11.1, R15.1
- new net +3V4: R13.2, R14.1, R17.2, R18.1, R20.1
- new net +6V8: R13.1, R17.1
- new net +8V4: R11.2, R12.1, R15.2, R16.1, R19.1
- new net GND: R12.2, R14.2, R16.2, R18.2, R19.2, R20.2
Other:
- note added: "I_{R1} = (U_{in} - U_{out}) / R1 = (12.7 - 8.4) / 220 = 0.0195A I_{R_{out}} = 0.007A R_{out} = U_{out} / I_{R_{out}} = 8.4 / 0.007 = 1200 I_{R2} = I_{R1} - I_{R_{out}} = 0.0195 - 0.007 = 0.0125A R2 = U_{out} / I_{R2} = 8.4 / 0.0125 = 672 -> 680"
- note added: "I_{R1} = (U_{in} - U_{out}) / R1 = (12.7 - 8.4) / 220 = 0.0195A R2 = U_{out} / I_{R1} = 8.4 / 0.0195 = 430"
- note added: "I_{R1} = (U_{in} - U_{out}) / R1 = (5.8 - 3.4) / 82 = 0.029A R2 = U_{out} / I_{R1} = 3.4 / 0.029 = 117 -> 120"
- note added: "I_{R1} = (U_{in} - U_{out}) / R1 = (6.8 - 3.4) / 82 = 0.041A I_{R_{out}} = 0.007A R_{out} = U_{out} / I_{R_{out}} = 3.4 / 0.007 = 485,71 I_{R2} = I_{R1} - I_{R_{out}} = 0.041 - 0.007 = 0.034A R2 = U_{out} / I_{R2} = 3.4 / 0.034 = 100 -> 100"
- note added: "Задача 2 - Рассчитать номиналы резисторов для делителя: из напряжения 12,7 В требуется получить на выходе 8,4 В при номинале резистора R1 220 Ом - Рассчитать номиналы резисторов для делителя: из напряжения 6,8 В требуется получить на выходе 3,4 В при номинале резистора R1 82 Ом - Произвести перерасчет делителей задач 2.1 и 2.2 при условии тока нагрузки, подключенной к выходу равной 7 мА. Номинал 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"

Commit message: home works 3 and 4
Parts:
- R17: renamed from R14; value ? -> 91
- renumbered R15 to R13, R16 to R14, R19 to R15, R13 to R16, R17 to R18, R18 to R19
Other:
- note added: "I_{R11} = (U_{in} - U_{out}) / R11 = (12.7 - 8.4) / 220 = 0.0195A R12 = U_{out} / I_{R11} = 8.4 / 0.0195 = 430"
- note added: "I_{R13} = (U_{in} - U_{out}) / R13 = (12.7 - 8.4) / 220 = 0.0195A I_{R15} = 0.007A R15 = U_{out} / I_{R15} = 8.4 / 0.007 = 1200 I_{R14} = I_{R13} - I_{R15} = 0.0195 - 0.007 = 0.0125A R14 = U_{out} / I_{R14} = 8.4 / 0.0125 = 672 -> 680"
- note added: "I_{R16} = (U_{in} - U_{out}) / R16 = (6.8 - 3.4) / 82 = 0.041A R17 = U_{out} / I_{R16} = 3.4 / 0.041 = 83 -> 91"
- note added: "I_{R18} = (U_{in} - U_{out}) / R18 = (6.8 - 3.4) / 82 = 0.041A I_{R20} = 0.007A R20 = U_{out} / I_{R20} = 3.4 / 0.007 = 485,71 I_{R19} = I_{R18} - I_{R20} = 0.041 - 0.007 = 0.034A R19 = U_{out} / I_{R20} = 3.4 / 0.034 = 100 -> 100"
- note removed: "I_{R1} = (U_{in} - U_{out}) / R1 = (12.7 - 8.4) / 220 = 0.0195A I_{R_{out}} = 0.007A R_{out} = U_{out} / I_{R_{out}} = 8.4 / 0.007 = 1200 I_{R2} = I_{R1} - I_{R_{out}} = 0.0195 - 0.007 = 0.0125A R2 = U_{out} / I_{R2} = 8.4 / 0.0125 = 672 -> 680"
- note removed: "I_{R1} = (U_{in} - U_{out}) / R1 = (12.7 - 8.4) / 220 = 0.0195A R2 = U_{out} / I_{R1} = 8.4 / 0.0195 = 430"
- note removed: "I_{R1} = (U_{in} - U_{out}) / R1 = (5.8 - 3.4) / 82 = 0.029A R2 = U_{out} / I_{R1} = 3.4 / 0.029 = 117 -> 120"
- note removed: "I_{R1} = (U_{in} - U_{out}) / R1 = (6.8 - 3.4) / 82 = 0.041A I_{R_{out}} = 0.007A R_{out} = U_{out} / I_{R_{out}} = 3.4 / 0.007 = 485,71 I_{R2} = I_{R1} - I_{R_{out}} = 0.041 - 0.007 = 0.034A R2 = U_{out} / I_{R2} = 3.4 / 0.034 = 100 -> 100"
- moved on the sheet: R11, R12, R13, R14, R15, R16, R17, R18, R19, R20
