File: home works/home work 03/task 03.kicad_sch (KiCad schematic)
At the start: 0 parts

Commit message: home work 3
Other:
- note added: "R = 1.8 кОм C = 0.47 нФ τ = R * C = 1.8 Ом * 0.47 нФ = 0.846 мкс зарядка до 95% = 3τ = 2.538 мкс"
- note added: "R = 6.8 Ом C = 33 мкФ τ = R * C = 6.8 * 33 мкФ = 224.4 мс зарядка до 95% = 3τ = 673.2 мс"
- note added: "R = 82 Ом C = 2.2 мкФ τ = R * C = 82 * 0.0000022 = 180.4 мс зарядка до 95% = 3τ = 541.2 мс"
- note added: "Задача 3 - Произвести расчет времени заряда конденсатора до 95%: - 2,2 мкФ, при сопротивлении 82 Ом; - 33 мкФ, при сопротивлении 6,8 Ом; - 0,47 нФ, при сопротивлении 1,8 кОм."
Changed lines of the file:
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@@
 	(generator_version "8.0")
 	(paper "A4")
+	(text "R = 1.8 кОм\nC = 0.47 нФ\n\nτ = R * C = 1.8 Ом * 0.47 нФ = 0.846 мкс\n\nзарядка до 95% = 3τ = 2.538 мкс"
+		(exclude_from_sim no)
+		(at 152.908 51.308 0)
+		(effects
+			(font
+				(size 1.27 1.27)
+			)
+			(justify left top)
+		)
+	)
+	(text "R = 82 Ом\nC = 2.2 мкФ\n\nτ = R * C = 82 * 0.0000022 = 180.4 мс\n\nзарядка до 95% = 3τ = 541.2 мс"
+		(exclude_from_sim no)
+		(at 25.908 51.308 0)
+		(effects
+			(font
+				(size 1.27 1.27)
+			)
+			(justify left top)
+		)
+	)
+	(text "Задача 3 \n- Произвести расчет времени заряда конденсатора до 95%:\n  - 2,2 мкФ, при сопротивлении 82 Ом;\n  - 33 мкФ, при сопротивлении 6,8 Ом;\n  - 0,47 нФ, при сопротивлении 1,8 кОм."
+		(exclude_from_sim no)
+		(at 25.146 25.908 0)
+		(effects
+			(font
+				(size 1.27 1.27)
+			)
+			(justify left top)
+		)
+	)
+	(text "R = 6.8 Ом\nC = 33 мкФ\n\nτ = R * C = 6.8 * 33 мкФ = 224.4 мс\n\nзарядка до 95% = 3τ = 673.2 мс"
+		(exclude_from_sim no)
+		(at 89.408 51.308 0)
+		(effects
+			(font
+				(size 1.27 1.27)
+			)
+			(justify left top)
+		)
+	)
 )

Commit message: home works 3 and 4
Changed lines of the file:
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@@
 	(text "Задача 3 \n- Произвести расчет времени заряда конденсатора до 95%:\n  - 2,2 мкФ, при сопротивлении 82 Ом;\n  - 33 мкФ, при сопротивлении 6,8 Ом;\n  - 0,47 нФ, при сопротивлении 1,8 кОм."
 		(exclude_from_sim no)
-		(at 25.146 25.908 0)
+		(at 25.908 25.654 0)
 		(effects
 			(font
