File: .home_works/home work 03.kicad_sch (KiCad schematic)
At the start: 0 parts

Commit message: rename folder to hidden
Other:
- sheet Задача 1: file ./home work 03/task 01.kicad_sch -> home work 03/task 01.kicad_sch
- sheet Задача 2: file ./home work 03/task 02.kicad_sch -> home work 03/task 02.kicad_sch
- sheet Задача 3: file ./home work 03/task 03.kicad_sch -> home work 03/task 03.kicad_sch
Changed lines of the file:
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@@
 			)
 		)
-		(property "Sheetfile" "./home work 03/task 01.kicad_sch"
+		(property "Sheetfile" "home work 03/task 01.kicad_sch"
 			(at 24.13 89.4846 0)
 			(effects
@@
 			)
 		)
-		(property "Sheetfile" "./home work 03/task 03.kicad_sch"
+		(property "Sheetfile" "home work 03/task 03.kicad_sch"
 			(at 128.27 89.4846 0)
 			(effects
@@
 			)
 		)
-		(property "Sheetfile" "./home work 03/task 02.kicad_sch"
+		(property "Sheetfile" "home work 03/task 02.kicad_sch"
 			(at 76.2 89.4846 0)
 			(effects
@@
 		)
 	)
-	(sheet_instances
-		(path "/"
-			(page "1")
-		)
-	)
