File: .home_works/home work 02.kicad_sch (KiCad schematic)
At the start: 4 parts, among them U1 AW9523B, U2 BL0910, U3 HLK-7628N, U4 XS2184

Commit message: update hw2
Parts:
- renumbered U4 to U3, U3 to U4
Other:
- moved on the sheet: U2, U3, U4
Changed lines of the file:
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@@
 	(symbol
 		(lib_id "mipt:XS2184")
-		(at 45.72 143.51 0)
+		(at 45.72 142.24 0)
 		(unit 1)
 		(exclude_from_sim no)
@@
 		(on_board yes)
 		(dnp no)
-		(property "Reference" "U4"
-			(at 59.436 107.95 0)
+		(property "Reference" "U3"
+			(at 59.436 106.68 0)
 			(effects
 				(font
@@
 		)
 		(property "Value" "XS2184"
-			(at 59.182 104.394 0)
+			(at 59.182 103.124 0)
 			(effects
 				(font
@@
 		)
 		(property "Footprint" "mipt:QFN-48-1EP_7x7mm_P0.5mm_EP5.6x5.6mm_1"
-			(at 45.72 143.51 0)
+			(at 45.72 142.24 0)
 			(effects
 				(font
@@
 		)
 		(property "Datasheet" "./datasheets/XS2184 Datasheet CN V1.0.pdf"
-			(at 85.598 112.014 0)
+			(at 85.598 110.744 0)
 			(effects
 				(font
@@
 		)
 		(property "Description" ""
-			(at 45.72 143.51 0)
+			(at 45.72 142.24 0)
 			(effects
 				(font
@@
 			(project "mipt"
 				(path "/34d483ea-61c1-4e08-b30a-5dee616d4777/c73feff7-a444-4fc1-b029-86822a883591"
-					(reference "U4")
+					(reference "U3")
 					(unit 1)
 				)
@@
 	(symbol
 		(lib_id "mipt:HLK-7628N")
-		(at 130.81 142.24 0)
+		(at 128.27 125.73 0)
 		(unit 1)
 		(exclude_from_sim no)
@@
 		(dnp no)
 		(fields_autoplaced yes)
-		(property "Reference" "U3"
-			(at 172.72 140.9699 0)
+		(property "Reference" "U4"
+			(at 170.18 124.4599 0)
 			(effects
 				(font
@@
 		)
 		(property "Value" "HLK-7628N"
-			(at 172.72 143.5099 0)
+			(at 170.18 126.9999 0)
 			(effects
 				(font
@@
 		)
 		(property "Footprint" "mipt:HLK-7628N"
-			(at 130.81 142.24 0)
+			(at 128.27 125.73 0)
 			(effects
 				(font
@@
 		)
 		(property "Datasheet" "./datasheets/HLK-7628N_V2.6.pdf"
-			(at 130.81 142.24 0)
+			(at 128.27 125.73 0)
 			(effects
 				(font
@@
 		)
 		(property "Description" ""
-			(at 130.81 142.24 0)
+			(at 128.27 125.73 0)
 			(effects
 				(font
@@
 			(project "mipt"
 				(path "/34d483ea-61c1-4e08-b30a-5dee616d4777/c73feff7-a444-4fc1-b029-86822a883591"
-					(reference "U3")
+					(reference "U4")
 					(unit 1)
 				)
@@
 	(symbol
 		(lib_id "mipt:bl0910")
-		(at 105.41 57.15 0)
+		(at 105.41 55.88 0)
 		(unit 1)
 		(exclude_from_sim no)
@@
 		(fields_autoplaced yes)
 		(property "Reference" "U2"
-			(at 110.1441 22.86 0)
+			(at 110.1441 21.59 0)
 			(effects
 				(font
@@
 		)
 		(property "Value" "BL0910"
-			(at 110.1441 25.4 0)
+			(at 110.1441 24.13 0)
 			(effects
 				(font
@@
 		)
 		(property "Footprint" "Package_QFP:LQFP-48_7x7mm_P0.5mm"
-			(at 144.78 18.288 0)
+			(at 144.78 17.018 0)
 			(effects
 				(font
@@
 		)
 		(property "Datasheet" "./datasheets/bl0910.pdf"
-			(at 137.922 22.86 0)
+			(at 137.922 21.59 0)
 			(effects
 				(font
@@
 		)
 		(property "Description" ""
-			(at 105.41 57.15 0)
-			(effects
-				(font
+			(at 105.41 55.88 0)
+			(effects
+				(font

Commit message: some fixes and add hw 5
Connections:
- net at U3.21 (DRAIN3): now also U3.29 (DRAIN3), U3.30 (DRAIN3)
- net at U3.22 (DRAIN4): now also U3.25 (DRAIN4), U3.26 (DRAIN4)
- net at U3.32 (DRAIN2): now also U3.40 (DRAIN2)
- net at U3.35 (DRAIN1): now also U3.36 (DRAIN1), U3.39 (DRAIN1)
- no-connect marks 24 -> 162
