File: .home_works/home work 03/task 01.kicad_sch (KiCad schematic)
At the start: 29 parts

Commit message: rename folder to hidden
Parts:
- renumbered D5 to D?, D16 to D?, D8 to D?, D13 to D?, D14 to D?, D4 to D?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

Commit message: update hw3
Parts:
- gave numbers to parts that had none: 29
