File: .home_works/home work 03/task 02.kicad_sch (KiCad schematic)
At the start: 10 parts

Commit message: rename folder to hidden
Parts:
- renumbered R20 to R?, R15 to R?, R11 to R?, R19 to R?, R17 to R?, R14 to R?, R16 to R?, R12 to R?, R18 to R?, R13 to R?
Changed lines of the file:
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@@
 		(dnp no)
 		(fields_autoplaced yes)
-		(property "Reference" "#PWR016"
+		(property "Reference" "#PWR?"
 			(at 50.8 130.81 0)
 			(effects
@@
 			(project "mipt"
 				(path "/34d483ea-61c1-4e08-b30a-5dee616d4777/cfdf2a98-d53d-4979-9485-05dd773be1bb/ca31be19-098b-42b9-ad83-8f969410d312"
-					(reference "#PWR016")
+					(reference "#PWR?")
 					(unit 1)
 				)
@@
 		(dnp no)
 		(fields_autoplaced yes)
-		(property "Reference" "#PWR012"
+		(property "Reference" "#PWR?"
 			(at 38.1 90.17 0)
 			(effects
@@
 			(project "mipt"
 				(path "/34d483ea-61c1-4e08-b30a-5dee616d4777/cfdf2a98-d53d-4979-9485-05dd773be1bb/ca31be19-098b-42b9-ad83-8f969410d312"
-					(reference "#PWR012")
+					(reference "#PWR?")
 					(unit 1)
 				)
@@
 		(dnp no)
 		(fields_autoplaced yes)
-		(property "Reference" "R20"
+		(property "Reference" "R?"
 			(at 162.56 135.8899 0)
 			(effects
@@
 			(project "mipt"
 				(path "/34d483ea-61c1-4e08-b30a-5dee616d4777/cfdf2a98-d53d-4979-9485-05dd773be1bb/ca31be19-098b-42b9-ad83-8f969410d312"
-					(reference "R20")
+					(reference "R?")
 					(unit 1)
 				)
@@
 		(dnp no)
 		(fields_autoplaced yes)
-		(property "Reference" "R15"
+		(property "Reference" "R?"
 			(at 162.56 72.3899 0)
 			(effects
@@
 			(project "mipt"
 				(path "/34d483ea-61c1-4e08-b30a-5dee616d4777/cfdf2a98-d53d-4979-9485-05dd773be1bb/ca31be19-098b-42b9-ad83-8f969410d312"
-					(reference "R15")
+					(reference "R?")
 					(unit 1)
 				)
@@
 		(dnp no)
 		(fields_autoplaced yes)
-		(property "Reference" "R11"
+		(property "Reference" "R?"
 			(at 40.64 58.4199 0)
 			(effects
@@
 		)
 		(instances
-			(project ""
-				(path "/34d483ea-61c1-4e08-b30a-5dee616d4777/cfdf2a98-d53d-4979-9485-05dd773be1bb/ca31be19-098b-42b9-ad83-8f969410d312"
-					(reference "R11")
+			(project "mipt"
+				(path "/34d483ea-61c1-4e08-b30a-5dee616d4777/cfdf2a98-d53d-4979-9485-05dd773be1bb/ca31be19-098b-42b9-ad83-8f969410d312"
+					(reference "R?")
 					(unit 1)
 				)
@@
 		(dnp no)
 		(fields_autoplaced yes)
-		(property "Reference" "#PWR08"
+		(property "Reference" "#PWR?"
 			(at 38.1 54.61 0)
 			(effects
@@
 			(project "mipt"
 				(path "/34d483ea-61c1-4e08-b30a-5dee616d4777/cfdf2a98-d53d-4979-9485-05dd773be1bb/ca31be19-098b-42b9-ad83-8f969410d312"
-					(reference "#PWR08")
+					(reference "#PWR?")
 					(unit 1)
 				)
@@
 		(dnp no)
 		(fields_autoplaced yes)
-		(property "Reference" "R19"
+		(property "Reference" "R?"
 			(at 149.86 135.8899 0)
 			(effects
@@
 			(project "mipt"
 				(path "/34d483ea-61c1-4e08-b30a-5dee616d4777/cfdf2a98-d53d-4979-9485-05dd773be1bb/ca31be19-098b-42b9-ad83-8f969410d312"
-					(reference "R19")
+					(reference "R?")
 					(unit 1)
 				)
@@
 		(dnp no)
 		(fields_autoplaced yes)
-		(property "Reference" "#PWR015"
+		(property "Reference" "#PWR?"
 			(at 160.02 129.54 0)
 			(effects
@@
 			(project "mipt"
 				(path "/34d483ea-61c1-4e08-b30a-5dee616d4777/cfdf2a98-d53d-4979-9485-05dd773be1bb/ca31be19-098b-42b9-ad83-8f969410d312"
-					(reference "#PWR015")
+					(reference "#PWR?")
 					(unit 1)
 				)
@@
 		(dnp no)
 		(fields_autoplaced yes)
-		(property "Reference" "R17"
+		(property "Reference" "R?"
 			(at 40.64 137.1599 0)
 			(effects
@@
 			(project "mipt"
 				(path "/34d483ea-61c1-4e08-b30a-5dee616d4777/cfdf2a98-d53d-4979-9485-05dd773be1bb/ca31be19-098b-42b9-ad83-8f969410d312"
-					(reference "R17")
+					(reference "R?")
 					(unit 1)
 				)
@@
 		(dnp no)
 		(fields_autoplaced yes)
-		(property "Reference" "#PWR011"
+		(property "Reference" "#PWR?"
 			(at 147.32 88.9 0)
 			(effects
@@
 			(project "mipt"
 				(path "/34d483ea-61c1-4e08-b30a-5dee616d4777/cfdf2a98-d53d-4979-9485-05dd773be1bb/ca31be19-098b-42b9-ad83-8f969410d312"
-					(reference "#PWR011")
+					(reference "#PWR?")
 					(unit 1)
 				)
@@
 		(dnp no)
 		(fields_autoplaced yes)
-		(property "Reference" "#PWR014"
+		(property "Reference" "#PWR?"
 			(at 38.1 118.11 0)
 			(effects
@@
 			(project "mipt"
 				(path "/34d483ea-61c1-4e08-b30a-5dee616d4777/cfdf2a98-d53d-4979-9485-05dd773be1bb/ca31be19-098b-42b9-ad83-8f969410d312"
-					(reference "#PWR014")
+					(reference "#PWR?")
 					(unit 1)
 				)
@@
 		(dnp no)
 		(fields_autoplaced yes)
-		(property "Reference" "R14"
+		(property "Reference" "R?"
 			(at 149.86 72.3899 0)
 			(effects
@@
 			(project "mipt"
 				(path "/34d483ea-61c1-4e08-b30a-5dee616d4777/cfdf2a98-d53d-4979-9485-05dd773be1bb/ca31be19-098b-42b9-ad83-8f969410d312"
-					(reference "R14")
+					(reference "R?")
 					(unit 1)
 				)
@@
 		(dnp no)
 		(fields_autoplaced yes)
-		(property "Reference" "#PWR07"
+		(property "Reference" "#PWR?"
 			(at 147.32 53.34 0)
 			(effects
@@
 			(project "mipt"
 				(path "/34d483ea-61c1-4e08-b30a-5dee616d4777/cfdf2a98-d53d-4979-9485-05dd773be1bb/ca31be19-098b-42b9-ad83-8f969410d312"
-					(reference "#PWR07")
+					(reference "#PWR?")
 					(unit 1)
 				)
@@
 		(dnp no)
 		(fields_autoplaced yes)
-		(property "Reference" "R16"
+		(property "Reference" "R?"
 			(at 40.64 121.9199 0)
 			(effects
@@
 			(project "mipt"
 				(path "/34d483ea-61c1-4e08-b30a-5dee616d4777/cfdf2a98-d53d-4979-9485-05dd773be1bb/ca31be19-098b-42b9-ad83-8f969410d312"
-					(reference "R16")
+					(reference "R?")
 					(unit 1)
 				)
@@
 		(dnp no)
 		(fields_autoplaced yes)
-		(property "Reference" "#PWR010"
+		(property "Reference" "#PWR?"
 			(at 50.8 67.31 0)
 			(effects
@@
 		)
 		(instances
-			(project ""
-				(path "/34d483ea-61c1-4e08-b30a-5dee616d4777/cfdf2a98-d53d-4979-9485-05dd773be1bb/ca31be19-098b-42b9-ad83-8f969410d312"
-					(reference "#PWR010")
+			(project "mipt"
+				(path "/34d483ea-61c1-4e08-b30a-5dee616d4777/cfdf2a98-d53d-4979-9485-05dd773be1bb/ca31be19-098b-42b9-ad83-8f969410d312"
+					(reference "#PWR?")
 					(unit 1)
 				)
@@
 		(dnp no)
 		(fields_autoplaced yes)
-		(property "Reference" "R12"
+		(property "Reference" "R?"
 			(at 40.64 73.6599 0)
 			(effects
@@
 			(project "mipt"
 				(path "/34d483ea-61c1-4e08-b30a-5dee616d4777/cfdf2a98-d53d-4979-9485-05dd773be1bb/ca31be19-098b-42b9-ad83-8f969410d312"
-					(reference "R12")
+					(reference "R?")
 					(unit 1)
 				)
@@
 		(dnp no)
 		(fields_autoplaced yes)
-		(property "Reference" "#PWR09"
+		(property "Reference" "#PWR?"
 			(at 160.02 66.04 0)
 			(effects
@@
 			(project "mipt"
 				(path "/34d483ea-61c1-4e08-b30a-5dee616d4777/cfdf2a98-d53d-4979-9485-05dd773be1bb/ca31be19-098b-42b9-ad83-8f969410d312"
-					(reference "#PWR09")
+					(reference "#PWR?")
 					(unit 1)
 				)
@@
 		(dnp no)
 		(fields_autoplaced yes)
-		(property "Reference" "R18"
+		(property "Reference" "R?"
 			(at 149.86 120.6499 0)
 			(effects
@@
 			(project "mipt"
 				(path "/34d483ea-61c1-4e08-b30a-5dee616d4777/cfdf2a98-d53d-4979-9485-05dd773be1bb/ca31be19-098b-42b9-ad83-8f969410d312"
-					(reference "R18")
+					(reference "R?")
 					(unit 1)
 				)
@@
 		(dnp no)
 		(fields_autoplaced yes)
-		(property "Reference" "#PWR018"
+		(property "Reference" "#PWR?"
 			(at 38.1 153.67 0)
 			(effects
@@
 			(project "mipt"
 				(path "/34d483ea-61c1-4e08-b30a-5dee616d4777/cfdf2a98-d53d-4979-9485-05dd773be1bb/ca31be19-098b-42b9-ad83-8f969410d312"
-					(reference "#PWR018")
+					(reference "#PWR?")
 					(unit 1)
 				)
@@
 		(dnp no)
 		(fields_autoplaced yes)
-		(property "Reference" "R13"
+		(property "Reference" "R?"
 			(at 149.86 57.1499 0)
 			(effects
@@
 			(project "mipt"
 				(path "/34d483ea-61c1-4e08-b30a-5dee616d4777/cfdf2a98-d53d-4979-9485-05dd773be1bb/ca31be19-098b-42b9-ad83-8f969410d312"
-					(reference "R13")
+					(reference "R?")
 					(unit 1)
 				)
@@
 		(dnp no)
 		(fields_autoplaced yes)
-		(property "Reference" "#PWR017"
+		(property "Reference" "#PWR?"
 			(at 147.32 152.4 0)
 			(effects
@@
 			(project "mipt"
 				(path "/34d483ea-61c1-4e08-b30a-5dee616d4777/cfdf2a98-d53d-4979-9485-05dd773be1bb/ca31be19-098b-42b9-ad83-8f969410d312"
-					(reference "#PWR017")
+					(reference "#PWR?")
 					(unit 1)
 				)
@@
 		(dnp no)
 		(fields_autoplaced yes)
-		(property "Reference" "#PWR013"
+		(property "Reference" "#PWR?"
 			(at 147.32 116.84 0)
 			(effects
@@
 			(project "mipt"
 				(path "/34d483ea-61c1-4e08-b30a-5dee616d4777/cfdf2a98-d53d-4979-9485-05dd773be1bb/ca31be19-098b-42b9-ad83-8f969410d312"
-					(reference "#PWR013")
-					(unit 1)
-				)
+					(reference "#PWR?")
+					(unit 1)
+				)

Commit message: update hw3
Parts:
- gave numbers to parts that had none: 10
Changed lines of the file:
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@@
 		(dnp no)
 		(fields_autoplaced yes)
-		(property "Reference" "R?"
+		(property "Reference" "R20"
 			(at 162.56 135.8899 0)
 			(effects
@@
 			(project "mipt"
 				(path "/34d483ea-61c1-4e08-b30a-5dee616d4777/cfdf2a98-d53d-4979-9485-05dd773be1bb/ca31be19-098b-42b9-ad83-8f969410d312"
-					(reference "R?")
+					(reference "R20")
 					(unit 1)
 				)
@@
 		(dnp no)
 		(fields_autoplaced yes)
-		(property "Reference" "R?"
+		(property "Reference" "R15"
 			(at 162.56 72.3899 0)
 			(effects
@@
 			(project "mipt"
 				(path "/34d483ea-61c1-4e08-b30a-5dee616d4777/cfdf2a98-d53d-4979-9485-05dd773be1bb/ca31be19-098b-42b9-ad83-8f969410d312"
-					(reference "R?")
+					(reference "R15")
 					(unit 1)
 				)
@@
 		(dnp no)
 		(fields_autoplaced yes)
-		(property "Reference" "R?"
+		(property "Reference" "R11"
 			(at 40.64 58.4199 0)
 			(effects
@@
 			(project "mipt"
 				(path "/34d483ea-61c1-4e08-b30a-5dee616d4777/cfdf2a98-d53d-4979-9485-05dd773be1bb/ca31be19-098b-42b9-ad83-8f969410d312"
-					(reference "R?")
+					(reference "R11")
 					(unit 1)
 				)
@@
 		(dnp no)
 		(fields_autoplaced yes)
-		(property "Reference" "R?"
+		(property "Reference" "R19"
 			(at 149.86 135.8899 0)
 			(effects
@@
 			(project "mipt"
 				(path "/34d483ea-61c1-4e08-b30a-5dee616d4777/cfdf2a98-d53d-4979-9485-05dd773be1bb/ca31be19-098b-42b9-ad83-8f969410d312"
-					(reference "R?")
+					(reference "R19")
 					(unit 1)
 				)
@@
 		(dnp no)
 		(fields_autoplaced yes)
-		(property "Reference" "R?"
+		(property "Reference" "R17"
 			(at 40.64 137.1599 0)
 			(effects
@@
 			(project "mipt"
 				(path "/34d483ea-61c1-4e08-b30a-5dee616d4777/cfdf2a98-d53d-4979-9485-05dd773be1bb/ca31be19-098b-42b9-ad83-8f969410d312"
-					(reference "R?")
+					(reference "R17")
 					(unit 1)
 				)
@@
 		(dnp no)
 		(fields_autoplaced yes)
-		(property "Reference" "R?"
+		(property "Reference" "R14"
 			(at 149.86 72.3899 0)
 			(effects
@@
 			(project "mipt"
 				(path "/34d483ea-61c1-4e08-b30a-5dee616d4777/cfdf2a98-d53d-4979-9485-05dd773be1bb/ca31be19-098b-42b9-ad83-8f969410d312"
-					(reference "R?")
+					(reference "R14")
 					(unit 1)
 				)
@@
 		(dnp no)
 		(fields_autoplaced yes)
-		(property "Reference" "R?"
+		(property "Reference" "R16"
 			(at 40.64 121.9199 0)
 			(effects
@@
 			(project "mipt"
 				(path "/34d483ea-61c1-4e08-b30a-5dee616d4777/cfdf2a98-d53d-4979-9485-05dd773be1bb/ca31be19-098b-42b9-ad83-8f969410d312"
-					(reference "R?")
+					(reference "R16")
 					(unit 1)
 				)
@@
 		(dnp no)
 		(fields_autoplaced yes)
-		(property "Reference" "R?"
+		(property "Reference" "R12"
 			(at 40.64 73.6599 0)
 			(effects
@@
 			(project "mipt"
 				(path "/34d483ea-61c1-4e08-b30a-5dee616d4777/cfdf2a98-d53d-4979-9485-05dd773be1bb/ca31be19-098b-42b9-ad83-8f969410d312"
-					(reference "R?")
+					(reference "R12")
 					(unit 1)
 				)
@@
 		(dnp no)
 		(fields_autoplaced yes)
-		(property "Reference" "R?"
+		(property "Reference" "R18"
 			(at 149.86 120.6499 0)
 			(effects
@@
 			(project "mipt"
 				(path "/34d483ea-61c1-4e08-b30a-5dee616d4777/cfdf2a98-d53d-4979-9485-05dd773be1bb/ca31be19-098b-42b9-ad83-8f969410d312"
-					(reference "R?")
+					(reference "R18")
 					(unit 1)
 				)
@@
 		(dnp no)
 		(fields_autoplaced yes)
-		(property "Reference" "R?"
+		(property "Reference" "R13"
 			(at 149.86 57.1499 0)
 			(effects
@@
 			(project "mipt"
 				(path "/34d483ea-61c1-4e08-b30a-5dee616d4777/cfdf2a98-d53d-4979-9485-05dd773be1bb/ca31be19-098b-42b9-ad83-8f969410d312"
-					(reference "R?")
-					(unit 1)
-				)
+					(reference "R13")
+					(unit 1)
+				)
