File: .home_works/home work 04/task 01.kicad_sch (KiCad schematic)
At the start: 5 parts, among them Q1 BC328, SW1 SW_Push

Commit message: rename folder to hidden
Parts:
- renumbered LA1 to LA?, Q1 to Q?, R22 to R?, R21 to R?, SW1 to SW?
Changed lines of the file:
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@@
 		(dnp no)
 		(fields_autoplaced yes)
-		(property "Reference" "SW1"
+		(property "Reference" "SW?"
 			(at 46.99 64.77 0)
 			(effects
@@
 		)
 		(instances
-			(project ""
-				(path "/34d483ea-61c1-4e08-b30a-5dee616d4777/f9b8cd78-f2f2-4446-aa11-838913d7a5bd/f08a2be2-cccb-4bdb-87b3-05d95f6eb5a2"
-					(reference "SW1")
+			(project "mipt"
+				(path "/34d483ea-61c1-4e08-b30a-5dee616d4777/f9b8cd78-f2f2-4446-aa11-838913d7a5bd/f08a2be2-cccb-4bdb-87b3-05d95f6eb5a2"
+					(reference "SW?")
 					(unit 1)
 				)
@@
 		(dnp no)
 		(fields_autoplaced yes)
-		(property "Reference" "R22"
+		(property "Reference" "R?"
 			(at 69.85 63.4999 0)
 			(effects
@@
 			(project "mipt"
 				(path "/34d483ea-61c1-4e08-b30a-5dee616d4777/f9b8cd78-f2f2-4446-aa11-838913d7a5bd/f08a2be2-cccb-4bdb-87b3-05d95f6eb5a2"
-					(reference "R22")
+					(reference "R?")
 					(unit 1)
 				)
@@
 		(dnp no)
 		(fields_autoplaced yes)
-		(property "Reference" "#PWR020"
+		(property "Reference" "#PWR?"
 			(at 78.74 57.15 0)
 			(effects
@@
 		)
 		(instances
-			(project ""
-				(path "/34d483ea-61c1-4e08-b30a-5dee616d4777/f9b8cd78-f2f2-4446-aa11-838913d7a5bd/f08a2be2-cccb-4bdb-87b3-05d95f6eb5a2"
-					(reference "#PWR020")
+			(project "mipt"
+				(path "/34d483ea-61c1-4e08-b30a-5dee616d4777/f9b8cd78-f2f2-4446-aa11-838913d7a5bd/f08a2be2-cccb-4bdb-87b3-05d95f6eb5a2"
+					(reference "#PWR?")
 					(unit 1)
 				)
@@
 		(dnp no)
 		(fields_autoplaced yes)
-		(property "Reference" "#PWR021"
+		(property "Reference" "#PWR?"
 			(at 78.74 101.6 0)
 			(effects
@@
 		)
 		(instances
-			(project ""
-				(path "/34d483ea-61c1-4e08-b30a-5dee616d4777/f9b8cd78-f2f2-4446-aa11-838913d7a5bd/f08a2be2-cccb-4bdb-87b3-05d95f6eb5a2"
-					(reference "#PWR021")
+			(project "mipt"
+				(path "/34d483ea-61c1-4e08-b30a-5dee616d4777/f9b8cd78-f2f2-4446-aa11-838913d7a5bd/f08a2be2-cccb-4bdb-87b3-05d95f6eb5a2"
+					(reference "#PWR?")
 					(unit 1)
 				)
@@
 		(dnp no)
 		(fields_autoplaced yes)
-		(property "Reference" "R21"
+		(property "Reference" "R?"
 			(at 59.69 66.04 90)
 			(effects
@@
 		)
 		(instances
-			(project ""
-				(path "/34d483ea-61c1-4e08-b30a-5dee616d4777/f9b8cd78-f2f2-4446-aa11-838913d7a5bd/f08a2be2-cccb-4bdb-87b3-05d95f6eb5a2"
-					(reference "R21")
+			(project "mipt"
+				(path "/34d483ea-61c1-4e08-b30a-5dee616d4777/f9b8cd78-f2f2-4446-aa11-838913d7a5bd/f08a2be2-cccb-4bdb-87b3-05d95f6eb5a2"
+					(reference "R?")
 					(unit 1)
 				)
@@
 		(dnp no)
 		(fields_autoplaced yes)
-		(property "Reference" "#PWR019"
+		(property "Reference" "#PWR?"
 			(at 38.1 57.15 0)
 			(effects
@@
 		)
 		(instances
-			(project ""
-				(path "/34d483ea-61c1-4e08-b30a-5dee616d4777/f9b8cd78-f2f2-4446-aa11-838913d7a5bd/f08a2be2-cccb-4bdb-87b3-05d95f6eb5a2"
-					(reference "#PWR019")
+			(project "mipt"
+				(path "/34d483ea-61c1-4e08-b30a-5dee616d4777/f9b8cd78-f2f2-4446-aa11-838913d7a5bd/f08a2be2-cccb-4bdb-87b3-05d95f6eb5a2"
+					(reference "#PWR?")
 					(unit 1)
 				)
@@
 		(on_board yes)
 		(dnp no)
-		(property "Reference" "Q1"
+		(property "Reference" "Q?"
 			(at 81.28 73.6601 0)
 			(effects
@@
 		)
 		(instances
-			(project ""
-				(path "/34d483ea-61c1-4e08-b30a-5dee616d4777/f9b8cd78-f2f2-4446-aa11-838913d7a5bd/f08a2be2-cccb-4bdb-87b3-05d95f6eb5a2"
-					(reference "Q1")
+			(project "mipt"
+				(path "/34d483ea-61c1-4e08-b30a-5dee616d4777/f9b8cd78-f2f2-4446-aa11-838913d7a5bd/f08a2be2-cccb-4bdb-87b3-05d95f6eb5a2"
+					(reference "Q?")
 					(unit 1)
 				)
@@
 		(dnp no)
 		(fields_autoplaced yes)
-		(property "Reference" "LA1"
+		(property "Reference" "LA?"
 			(at 82.55 85.0899 0)
 			(effects
@@
 		)
 		(instances
-			(project ""
-				(path "/34d483ea-61c1-4e08-b30a-5dee616d4777/f9b8cd78-f2f2-4446-aa11-838913d7a5bd/f08a2be2-cccb-4bdb-87b3-05d95f6eb5a2"
-					(reference "LA1")
-					(unit 1)
-				)
+			(project "mipt"
+				(path "/34d483ea-61c1-4e08-b30a-5dee616d4777/f9b8cd78-f2f2-4446-aa11-838913d7a5bd/f08a2be2-cccb-4bdb-87b3-05d95f6eb5a2"
+					(reference "LA?")
+					(unit 1)
+				)

Commit message: add hw 4
Parts:
- Q1: renamed from Q?; value BC328 -> BC327-40
- R21: renamed from R?; value 3 -> 3k3
- R22: renamed from R?; value 3 -> 33k
- gave numbers to parts that had none: 2
Connections:
- net +3.3V renamed -3.3V
Other:
- note added: "I_{C} = 250 mA V_{load} = +12V V_{control} = -3.3V hfe = 210 V_{CE_{sat}} = 0.7V V_{BE_{sat}} = 0.02V I_{C} = I_{B} * hfe I_{B} = 250 / 210 = 1.19 mA R_{B} = (V_{control} - V_{BE}) / I_{B} = (-3.3 - 0.7) / 0.00119 = -3361.34453782 Om = -3.36134453782 kOm -> 3k3 P = I_{C} * V_{CE} = 0.21 * 0.02 = 0.0042 Вт = 4 мВт"
- note added: "Задача 1 Рассчитать и выполнить подключение нагрузки через PNP транзистор. Нагрузкой является лампа накаливания из набора (напряжение лампы 12 В, ток измерить мультиметром) Управление включением производить тактовой кнопкой (кнопка нажата - лампа горит). Напряжение управляющего сигнала 3.3 В."
- note removed: "I_{C} = 100 mA V_{in} = +12V V_{control} = +3.3V hfe = 120 V_{BE} = 0.8V V_{CE} = 0.06V I_{C} = I_{B} * hfe I_{B} = 100 / 120 = 0.83 mA R_{B} = (V_{control} - V_{BE}) / I_{B} = (3.3 - 0.8) / 0.83 = 3.012 P = I_{C} * V_{CE} = 0.1 * 0.06 = 0.006 Вт = 6 мВт"
- note removed: "Задача 1 Рассчитать и выполнить подключение нагрузки через PNP транзистор. Нагрузкой является лампа накаливания из набора (напряжение лампы 12 В, ток измерить мультиметром) Управление включением производить тактовой кнопкой (кнопка нажата- лампа горит). Напряжение управляющего сигнала 3.3 В."
Changed lines of the file:
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@@
 		)
 	)
-	(text "Задача 1\nРассчитать и выполнить подключение нагрузки через PNP транзистор.\n\nНагрузкой является лампа накаливания из набора (напряжение лампы 12 В, ток измерить мультиметром)\n\nУправление включением производить тактовой кнопкой (кнопка нажата- лампа горит). Напряжение управляющего сигнала 3.3 В.\n"
+	(text "Задача 1\nРассчитать и выполнить подключение нагрузки через PNP транзистор.\n\nНагрузкой является лампа накаливания из набора (напряжение лампы 12 В, ток измерить мультиметром)\n\nУправление включением производить тактовой кнопкой (кнопка нажата - лампа горит). Напряжение управляющего сигнала 3.3 В.\n"
 		(exclude_from_sim no)
 		(at 25.4 25.654 0)
@@
 		)
 	)
-	(text "I_{C} = 100 mA\nV_{in} = +12V\nV_{control} = +3.3V\n\nhfe = 120\nV_{BE} = 0.8V\nV_{CE} = 0.06V\n\nI_{C} = I_{B} * hfe\nI_{B} = 100 / 120 = 0.83 mA\nR_{B} = (V_{control} - V_{BE}) / I_{B} = (3.3 - 0.8) / 0.83 = 3.012\n\nP = I_{C} * V_{CE} = 0.1 * 0.06 = 0.006 Вт = 6 мВт\n\n"
+	(text "I_{C} = 250 mA\nV_{load} = +12V\nV_{control} = -3.3V\n\nhfe = 210\nV_{CE_{sat}} = 0.7V\nV_{BE_{sat}} = 0.02V\n\nI_{C} = I_{B} * hfe\nI_{B} = 250 / 210 = 1.19 mA\nR_{B} = (V_{control} - V_{BE}) / I_{B} = (-3.3 - 0.7) / 0.00119 = -3361.34453782 Om = -3.36134453782 kOm -> 3k3\n\nP = I_{C} * V_{CE} = 0.21 * 0.02 = 0.0042 Вт = 4 мВт\n\n"
 		(exclude_from_sim no)
 		(at 101.6 51.308 0)
@@
 		(dnp no)
 		(fields_autoplaced yes)
-		(property "Reference" "SW?"
+		(property "Reference" "SW1"
 			(at 46.99 64.77 0)
 			(effects
@@
 			(project "mipt"
 				(path "/34d483ea-61c1-4e08-b30a-5dee616d4777/f9b8cd78-f2f2-4446-aa11-838913d7a5bd/f08a2be2-cccb-4bdb-87b3-05d95f6eb5a2"
-					(reference "SW?")
+					(reference "SW1")
 					(unit 1)
 				)
@@
 		(dnp no)
 		(fields_autoplaced yes)
-		(property "Reference" "R?"
+		(property "Reference" "R22"
 			(at 69.85 63.4999 0)
 			(effects
@@
 			)
 		)
-		(property "Value" "3"
+		(property "Value" "33k"
 			(at 69.85 66.0399 0)
 			(effects
@@
 			(project "mipt"
 				(path "/34d483ea-61c1-4e08-b30a-5dee616d4777/f9b8cd78-f2f2-4446-aa11-838913d7a5bd/f08a2be2-cccb-4bdb-87b3-05d95f6eb5a2"
-					(reference "R?")
+					(reference "R22")
 					(unit 1)
 				)
@@
 		(dnp no)
 		(fields_autoplaced yes)
-		(property "Reference" "R?"
+		(property "Reference" "R21"
 			(at 59.69 66.04 90)
 			(effects
@@
 			)
 		)
-		(property "Value" "3"
+		(property "Value" "3k3"
 			(at 59.69 68.58 90)
 			(effects
@@
 			(project "mipt"
 				(path "/34d483ea-61c1-4e08-b30a-5dee616d4777/f9b8cd78-f2f2-4446-aa11-838913d7a5bd/f08a2be2-cccb-4bdb-87b3-05d95f6eb5a2"
-					(reference "R?")
+					(reference "R21")
 					(unit 1)
 				)
@@
 			)
 		)
-		(property "Value" "+3.3V"
-			(at 38.1 48.26 0)
-			(effects
-				(font
-					(size 1.27 1.27)
-				)
+		(property "Value" "-3.3V"
+			(at 40.64 52.0699 0)
+			(effects
+				(font
+					(size 1.27 1.27)
+				)
+				(justify left)
 			)
 		)
@@
 		(on_board yes)
 		(dnp no)
-		(property "Reference" "Q?"
+		(property "Reference" "Q1"
 			(at 81.28 73.6601 0)
 			(effects
@@
 			)
 		)
-		(property "Value" "BC328"
+		(property "Value" "BC327-40"
 			(at 81.28 71.1201 0)
 			(effects
@@
 			(project "mipt"
 				(path "/34d483ea-61c1-4e08-b30a-5dee616d4777/f9b8cd78-f2f2-4446-aa11-838913d7a5bd/f08a2be2-cccb-4bdb-87b3-05d95f6eb5a2"
-					(reference "Q?")
+					(reference "Q1")
 					(unit 1)
 				)
@@
 		(dnp no)
 		(fields_autoplaced yes)
-		(property "Reference" "LA?"
+		(property "Reference" "LA1"
 			(at 82.55 85.0899 0)
 			(effects
@@
 			(project "mipt"
 				(path "/34d483ea-61c1-4e08-b30a-5dee616d4777/f9b8cd78-f2f2-4446-aa11-838913d7a5bd/f08a2be2-cccb-4bdb-87b3-05d95f6eb5a2"
-					(reference "LA?")
-					(unit 1)
-				)
+					(reference "LA1")
+					(unit 1)
+				)
