File: .home_works/home work 04/task 02.kicad_sch (KiCad schematic)
At the start: 0 parts

Commit message: add hw 4
Parts:
- added LA2: Lamp, symbol Device:Lamp
- added Q2: BC337-40, Package_TO_SOT_THT:TO-92_Inline, symbol Transistor_BJT:BC337
- added R23: R_Photo, symbol Device:R_Photo
- added RV1: R_Potentiometer, symbol Device:R_Potentiometer
Connections:
- new net: Q2.2 (B), R23.1, RV1.3
- new net: LA2.1 (-), Q2.1 (C)
- new net +12V: LA2.2 (+)
- new net +3.3V: RV1.1, RV1.2
- new net GND: Q2.3 (E), R23.2
