File: home_work_05/task_01.kicad_sch (KiCad schematic)
At the start: 7 parts

Commit message: do home work 5
Parts:
- removed BT?: Battery, symbol Device:Battery
- added J2: Screw_Terminal_01x02, mipt:FK301-5.0, symbol Connector:Screw_Terminal_01x02
- D1: renamed from D?; value LED -> Red
- gave numbers to parts that had none: 5
Connections:
- net GND: now reaches Q1.3 (E), RV1.3
- net GND: now also J2.2 (Pin_2)
- net +12V: now reaches BZ1.1 (+), D1.2 (A), J1.1 (Pin_1)
- net +12V: now also J2.1 (Pin_1)
