File: home_work_05/home_work.kicad_sch (KiCad schematic)
At the start: 0 parts

Commit message: do home work 5
Parts:
- added BZ?: Buzzer, Buzzer_Beeper:Buzzer_15x7.5RM7.6, symbol Device:Buzzer
- added D?: Red, LED_THT:LED_D5.0mm, symbol Device:LED
- added J?: Conn_01x02_Pin, Connector_JST:JST_PH_B2B-PH-K_1x02_P2.00mm_Vertical, symbol Connector:Conn_01x02_Pin
- added J?: Screw_Terminal_01x02, mipt:FK301-5.0, symbol Connector:Screw_Terminal_01x02
- added Q?: BC337-40, Package_TO_SOT_THT:TO-92_Inline, symbol Transistor_BJT:BC337
- added R?: R, Resistor_THT:R_Axial_DIN0207_L6.3mm_D2.5mm_P10.16mm_Horizontal, symbol Device:R
- added RV?: R_Potentiometer, Potentiometer_THT:Potentiometer_Bourns_3266Y_Vertical, symbol Device:R_Potentiometer
Connections:
- new net: BZ?.2 (-), Q?.1 (C)
- new net: D?.1 (K), J?.2 (Pin_2), R?.2, RV?.1, RV?.2
- new net: Q?.2 (B), R?.1
- new net +12V: BZ?.1 (+), D?.2 (A), J?.1 (Pin_1), J?.1 (Pin_1)
- new net GND: J?.2 (Pin_2), Q?.3 (E), RV?.3
Other:
- removed sheet Задача 1

Commit message: update pcb and footprint
Connections:
- net +12V renamed +5V
Changed lines of the file:
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@@
 			)
 		)
-		(property "Value" "+12V"
-			(at 123.19 54.61 0)
-			(effects
-				(font
-					(size 1.27 1.27)
-				)
+		(property "Value" "+5V"
+			(at 125.73 58.4199 0)
+			(effects
+				(font
+					(size 1.27 1.27)
+				)
+				(justify left)
 			)
 		)
@@
 			)
 		)
-		(property "Value" "+12V"
-			(at 99.06 54.61 0)
-			(effects
-				(font
-					(size 1.27 1.27)
-				)
-			)
-		)
+		(property "Value" "+5V"
+			(at 101.6 58.4199 0)
+			(effects
+				(font
+					(size 1.27 1.27)
+				)
+				(justify left)
+			)
+		)

Commit message: do home work 5
Parts:
- gave numbers to parts that had none: 7
Changed lines of the file:
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@@
 		(dnp no)
 		(fields_autoplaced yes)
-		(property "Reference" "BZ?"
+		(property "Reference" "BZ1"
 			(at 105.41 68.5799 0)
 			(effects
@@
 			(project "home_work"
 				(path "/2dc85d6d-5070-4742-814b-83a7bb72a5d3"
-					(reference "BZ?")
+					(reference "BZ1")
 					(unit 1)
 				)
@@
 		(dnp no)
 		(fields_autoplaced yes)
-		(property "Reference" "J?"
+		(property "Reference" "J1"
 			(at 50.165 64.77 0)
 			(effects
@@
 			(project "home_work"
 				(path "/2dc85d6d-5070-4742-814b-83a7bb72a5d3"
-					(reference "J?")
+					(reference "J1")
 					(unit 1)
 				)
@@
 		(dnp no)
 		(fields_autoplaced yes)
-		(property "Reference" "Q?"
+		(property "Reference" "Q1"
 			(at 101.6 80.0099 0)
 			(effects
@@
 			(project "home_work"
 				(path "/2dc85d6d-5070-4742-814b-83a7bb72a5d3"
-					(reference "Q?")
+					(reference "Q1")
 					(unit 1)
 				)
@@
 		(dnp no)
 		(fields_autoplaced yes)
-		(property "Reference" "RV?"
+		(property "Reference" "RV1"
 			(at 55.88 91.4399 0)
 			(effects
@@
 			(project "home_work"
 				(path "/2dc85d6d-5070-4742-814b-83a7bb72a5d3"
-					(reference "RV?")
+					(reference "RV1")
 					(unit 1)
 				)
@@
 		(dnp no)
 		(fields_autoplaced yes)
-		(property "Reference" "D?"
+		(property "Reference" "D1"
 			(at 72.39 71.4374 90)
 			(effects
@@
 			(project "home_work"
 				(path "/2dc85d6d-5070-4742-814b-83a7bb72a5d3"
-					(reference "D?")
+					(reference "D1")
 					(unit 1)
 				)
@@
 		(dnp no)
 		(fields_autoplaced yes)
-		(property "Reference" "R?"
+		(property "Reference" "R1"
 			(at 83.82 74.93 90)
 			(effects
@@
 			(project "home_work"
 				(path "/2dc85d6d-5070-4742-814b-83a7bb72a5d3"
-					(reference "R?")
+					(reference "R1")
 					(unit 1)
 				)
@@
 		(dnp no)
 		(fields_autoplaced yes)
-		(property "Reference" "J?"
+		(property "Reference" "J2"
 			(at 134.62 63.4999 0)
 			(effects
@@
 			(project "home_work"
 				(path "/2dc85d6d-5070-4742-814b-83a7bb72a5d3"
-					(reference "J?")
-					(unit 1)
-				)
+					(reference "J2")
+					(unit 1)
+				)

Commit message: update home work 05
Parts:
- R1: value R -> 33K
- RV1: value R_Potentiometer -> 1M
Changed lines of the file:
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@@
 			)
 		)
-		(property "Value" "R_Potentiometer"
+		(property "Value" "1M"
 			(at 55.88 93.9799 0)
 			(effects
@@
 			)
 		)
-		(property "Value" "R"
+		(property "Value" "33K"
 			(at 83.82 77.47 90)
 			(effects
