File: home_work_04/task_01.kicad_sch (KiCad schematic)
At the start: 5 parts, among them Q1 BC327-40, SW1 SW_Push

Commit message: update home work 04
Parts:
- added BT1: 3.3V, symbol Device:Battery
- added BT2: 12V, symbol Device:Battery
Connections:
- net +12V: no longer names the net of Q1.3 (E), R2.2
- net +12V: now also BT1.1 (+), BT2.1 (+)
- net -3.3V: no longer names the net of SW1.1
- net -3.3V: now also BT1.2 (-)
- net GND: no longer names the net of LA1.1 (-)
- net GND: now also BT2.2 (-)
Other:
- note added: "I_{C} = 250 mA V_{BT2} = +12V V_{BT1} = -3.3V hfe = 210 V_{CE_{sat}} = 0.7V V_{BE_{sat}} = 0.02V I_{C} = I_{B} * hfe I_{B} = 250 / 210 = 1.19 mA R_{B} = (V_{control} - V_{BE}) / I_{B} = (-3.3 - 0.7) / 0.00119 = -3361.34453782 Om = -3.36134453782 kOm -> 3k3 P = I_{C} * V_{CE} = 0.21 * 0.02 = 0.0042 Вт = 4 мВт"
- note removed: "I_{C} = 250 mA V_{load} = +12V V_{control} = -3.3V hfe = 210 V_{CE_{sat}} = 0.7V V_{BE_{sat}} = 0.02V I_{C} = I_{B} * hfe I_{B} = 250 / 210 = 1.19 mA R_{B} = (V_{control} - V_{BE}) / I_{B} = (-3.3 - 0.7) / 0.00119 = -3361.34453782 Om = -3.36134453782 kOm -> 3k3 P = I_{C} * V_{CE} = 0.21 * 0.02 = 0.0042 Вт = 4 мВт"
- moved on the sheet: LA1, Q1, R1, R2, SW1

Commit message: update home work 04
Parts:
- R1: value 3k3 -> 7k5
- R2: value 33k -> 75k
Other:
- note added: "I_{C} = 250 mA V_{BT2} = 12V V_{BT1} = 3.3V hfe = 210 V_{CE_{sat}} = 0.85V V_{BE_{sat}} = 0.12V I_{C} = I_{B} * hfe I_{B} = 250 / 210 = 1.19 mA R_{B} = (V_{load} - V_{control} - V_{BE}) / I_{B} = (12 - 3.3 - 0.12) / 0.00119 = 7210.0840336134 Om = 7.2100840336134 kOm -> 7k5 P = (I_{C} * V_{CE}) + (I_{B} * V_{BE}) = (0.25 * 0.85) + (0.00119 * 0.12) = 0.2125 + 0.0001428 = 0.2126428 = 2,1 мВт"
- note added: "https://tinyurl.com/2aj4gmdg"
- note removed: "I_{C} = 250 mA V_{BT2} = +12V V_{BT1} = -3.3V hfe = 210 V_{CE_{sat}} = 0.7V V_{BE_{sat}} = 0.02V I_{C} = I_{B} * hfe I_{B} = 250 / 210 = 1.19 mA R_{B} = (V_{control} - V_{BE}) / I_{B} = (-3.3 - 0.7) / 0.00119 = -3361.34453782 Om = -3.36134453782 kOm -> 3k3 P = I_{C} * V_{CE} = 0.21 * 0.02 = 0.0042 Вт = 4 мВт"
Changed lines of the file:
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@@
 		)
 	)
-	(text "I_{C} = 250 mA\nV_{BT2} = +12V\nV_{BT1} = -3.3V\n\nhfe = 210\nV_{CE_{sat}} = 0.7V\nV_{BE_{sat}} = 0.02V\n\nI_{C} = I_{B} * hfe\nI_{B} = 250 / 210 = 1.19 mA\nR_{B} = (V_{control} - V_{BE}) / I_{B} = (-3.3 - 0.7) / 0.00119 = -3361.34453782 Om = -3.36134453782 kOm -> 3k3\n\nP = I_{C} * V_{CE} = 0.21 * 0.02 = 0.0042 Вт = 4 мВт\n\n"
+	(text "https://tinyurl.com/2aj4gmdg"
+		(exclude_from_sim no)
+		(at 60.706 106.426 0)
+		(effects
+			(font
+				(size 1.27 1.27)
+			)
+		)
+	)
+	(text "I_{C} = 250 mA\nV_{BT2} = 12V\nV_{BT1} = 3.3V\n\nhfe = 210\nV_{CE_{sat}} = 0.85V\nV_{BE_{sat}} = 0.12V\n\nI_{C} = I_{B} * hfe\n\nI_{B} = 250 / 210 = 1.19 mA\n\nR_{B} = (V_{load} - V_{control} - V_{BE}) / I_{B} \n      = (12 - 3.3 - 0.12) / 0.00119 = 7210.0840336134 Om \n      = 7.2100840336134 kOm -> 7k5\n\nP = (I_{C} * V_{CE}) + (I_{B} * V_{BE}) \n  = (0.25 * 0.85) + (0.00119 * 0.12)\n  = 0.2125 + 0.0001428 = 0.2126428 = 2,1 мВт\n\n"
 		(exclude_from_sim no)
 		(at 104.648 51.308 0)
@@
 			)
 		)
-		(property "Value" "33k"
+		(property "Value" "75k"
 			(at 63.5 62.2299 0)
 			(effects
@@
 			)
 		)
-		(property "Value" "3k3"
+		(property "Value" "7k5"
 			(at 53.34 64.77 90)
 			(effects

Commit message: fix home work 04
Parts:
- R1: value 7k5 -> 2k7
- R2: value 75k -> 27k
Other:
- note added: "I_{C} = 250 mA V_{BT2} = 12.21V V_{BT1} = 3.3V hfe = 210 V_{CE_{sat}} = 0.85V V_{BE_{sat}} = 0.12V I_{C} = I_{B} * hfe I_{B} = 250 / 210 = 1.19 mA R_{B} = (V_{load} - V_{control} - V_{BE}) / I_{B} = (3.3 - 0.12) / 0.00119 = 2672.268907563 Om = 2.672268907563 kOm -> 2k7 P = (I_{C} * V_{CE}) + (I_{B} * V_{BE}) = (0.25 * 0.85) + (0.00119 * 0.12) = 0.2125 + 0.0001428 = 0.2126428 = 2,1 мВт"
- note removed: "I_{C} = 250 mA V_{BT2} = 12V V_{BT1} = 3.3V hfe = 210 V_{CE_{sat}} = 0.85V V_{BE_{sat}} = 0.12V I_{C} = I_{B} * hfe I_{B} = 250 / 210 = 1.19 mA R_{B} = (V_{load} - V_{control} - V_{BE}) / I_{B} = (12 - 3.3 - 0.12) / 0.00119 = 7210.0840336134 Om = 7.2100840336134 kOm -> 7k5 P = (I_{C} * V_{CE}) + (I_{B} * V_{BE}) = (0.25 * 0.85) + (0.00119 * 0.12) = 0.2125 + 0.0001428 = 0.2126428 = 2,1 мВт"
Changed lines of the file:
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@@
 		)
 	)
-	(text "I_{C} = 250 mA\nV_{BT2} = 12V\nV_{BT1} = 3.3V\n\nhfe = 210\nV_{CE_{sat}} = 0.85V\nV_{BE_{sat}} = 0.12V\n\nI_{C} = I_{B} * hfe\n\nI_{B} = 250 / 210 = 1.19 mA\n\nR_{B} = (V_{load} - V_{control} - V_{BE}) / I_{B} \n      = (12 - 3.3 - 0.12) / 0.00119 = 7210.0840336134 Om \n      = 7.2100840336134 kOm -> 7k5\n\nP = (I_{C} * V_{CE}) + (I_{B} * V_{BE}) \n  = (0.25 * 0.85) + (0.00119 * 0.12)\n  = 0.2125 + 0.0001428 = 0.2126428 = 2,1 мВт\n\n"
+	(text "I_{C} = 250 mA\nV_{BT2} = 12.21V\nV_{BT1} = 3.3V\n\nhfe = 210\nV_{CE_{sat}} = 0.85V\nV_{BE_{sat}} = 0.12V\n\nI_{C} = I_{B} * hfe\n\nI_{B} = 250 / 210 = 1.19 mA\n\nR_{B} = (V_{load} - V_{control} - V_{BE}) / I_{B} \n      = (3.3 - 0.12) / 0.00119 = 2672.268907563 Om \n      = 2.672268907563 kOm -> 2k7\n\nP = (I_{C} * V_{CE}) + (I_{B} * V_{BE}) \n  = (0.25 * 0.85) + (0.00119 * 0.12)\n  = 0.2125 + 0.0001428 = 0.2126428 = 2,1 мВт\n\n"
 		(exclude_from_sim no)
 		(at 104.648 51.308 0)
@@
 			)
 		)
-		(property "Value" "75k"
+		(property "Value" "27k"
 			(at 63.5 62.2299 0)
 			(effects
@@
 			)
 		)
-		(property "Value" "7k5"
+		(property "Value" "2k7"
 			(at 53.34 64.77 90)
 			(effects
