File: home_work_04/task_02.kicad_sch (KiCad schematic)
At the start: 4 parts, among them Q2 BC337-40

Commit message: update home work 04
Parts:
- added R4: 2K2, symbol Device:R
- R3: value R_Photo -> 1M
- RV1: value R_Potentiometer -> 1M
Connections:
- net at R3.1, RV1.3: now also R4.1; no longer Q2.2 (B)
- new net: Q2.2 (B), R4.2
Other:
- note added: "V_{control} = 3.3V V_{load} = 12V I_{C} = 250mA hfe = 220 I_{B} = I_{C} / hfe = 250 / 220 = 1.14 mA V_{BE} = 0.85V R_{B} = (V_{control} - V_{BE}) / I_{B} = (3.3 - 0.85) / 0.00114 = 2150 Om - 2K2"
- moved on the sheet: R3, RV1
Changed lines of the file:
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@@
 	(paper "A4")
 	(junction
-		(at 67.31 77.47)
+		(at 59.69 77.47)
 		(diameter 0)
 		(color 0 0 0 0)
 	)
 	(junction
-		(at 67.31 58.42)
+		(at 59.69 58.42)
 		(diameter 0)
 		(color 0 0 0 0)
@@
 	(wire
 		(pts
-			(xy 67.31 88.9) (xy 67.31 92.71)
+			(xy 59.69 77.47) (xy 59.69 81.28)
+		)
+		(stroke
+			(width 0)
+			(type default)
+		)
+	)
+	(wire
+		(pts
+			(xy 59.69 88.9) (xy 59.69 92.71)
 		)
 		(stroke
@@
 	(wire
 		(pts
-			(xy 67.31 77.47) (xy 78.74 77.47)
+			(xy 74.93 77.47) (xy 78.74 77.47)
 		)
 		(stroke
@@
 	(wire
 		(pts
-			(xy 67.31 58.42) (xy 67.31 62.23)
-		)
-		(stroke
-			(width 0)
-			(type default)
-		)
-	)
-	(wire
-		(pts
-			(xy 67.31 54.61) (xy 67.31 58.42)
-		)
-		(stroke
-			(width 0)
-			(type default)
-		)
-	)
-	(wire
-		(pts
-			(xy 67.31 77.47) (xy 67.31 81.28)
-		)
-		(stroke
-			(width 0)
-			(type default)
-		)
-	)
-	(wire
-		(pts
-			(xy 71.12 66.04) (xy 74.93 66.04)
-		)
-		(stroke
-			(width 0)
-			(type default)
-		)
-	)
-	(wire
-		(pts
-			(xy 74.93 66.04) (xy 74.93 58.42)
-		)
-		(stroke
-			(width 0)
-			(type default)
-		)
-	)
-	(wire
-		(pts
-			(xy 67.31 58.42) (xy 74.93 58.42)
-		)
-		(stroke
-			(width 0)
-			(type default)
-		)
-	)
-	(wire
-		(pts
-			(xy 67.31 69.85) (xy 67.31 77.47)
-		)
-		(stroke
-			(width 0)
-			(type default)
+			(xy 59.69 58.42) (xy 59.69 62.23)
+		)
+		(stroke
+			(width 0)
+			(type default)
+		)
+	)
+	(wire
+		(pts
+			(xy 59.69 77.47) (xy 67.31 77.47)
+		)
+		(stroke
+			(width 0)
+			(type default)
+		)
+	)
+	(wire
+		(pts
+			(xy 59.69 54.61) (xy 59.69 58.42)
+		)
+		(stroke
+			(width 0)
+			(type default)
+		)
+	)
+	(wire
+		(pts
+			(xy 63.5 66.04) (xy 67.31 66.04)
+		)
+		(stroke
+			(width 0)
+			(type default)
+		)
+	)
+	(wire
+		(pts
+			(xy 67.31 66.04) (xy 67.31 58.42)
+		)
+		(stroke
+			(width 0)
+			(type default)
+		)
+	)
+	(wire
+		(pts
+			(xy 59.69 58.42) (xy 67.31 58.42)
+		)
+		(stroke
+			(width 0)
+			(type default)
+		)
+	)
+	(wire
+		(pts
+			(xy 59.69 69.85) (xy 59.69 77.47)
+		)
+		(stroke
+			(width 0)
+			(type default)
+		)
+	)
+	(text "V_{control} = 3.3V\nV_{load} = 12V\nI_{C} = 250mA\nhfe = 220\nI_{B} = I_{C} / hfe = 250 / 220 =  1.14 mA\nV_{BE} = 0.85V\nR_{B} = (V_{control} - V_{BE}) / I_{B} = (3.3 - 0.85) / 0.00114 = 2150 Om - 2K2\n"
+		(exclude_from_sim no)
+		(at 114.554 51.308 0)
+		(effects
+			(font
+				(size 1.27 1.27)
+			)
+			(justify left top)
 		)
 	)
@@
 	(symbol
 		(lib_id "Device:R_Potentiometer")
-		(at 67.31 66.04 0)
+		(at 59.69 66.04 0)
 		(unit 1)
 		(exclude_from_sim no)
@@
 		(fields_autoplaced yes)
 		(property "Reference" "RV1"
-			(at 64.77 64.7699 0)
+			(at 57.15 64.7699 0)
 			(effects
 				(font
@@
 			)
 		)
-		(property "Value" "R_Potentiometer"
-			(at 64.77 67.3099 0)
+		(property "Value" "1M"
+			(at 57.15 67.3099 0)
 			(effects
 				(font
@@
 		)
 		(property "Footprint" ""
-			(at 67.31 66.04 0)
+			(at 59.69 66.04 0)
 			(effects
 				(font
@@
 		)
 		(property "Datasheet" "~"
-			(at 67.31 66.04 0)
+			(at 59.69 66.04 0)
 			(effects
 				(font
@@
 		)
 		(property "Description" "Potentiometer"
-			(at 67.31 66.04 0)
+			(at 59.69 66.04 0)
 			(effects
 				(font
@@
 	)
 	(symbol
+		(lib_id "Device:R")
+		(at 71.12 77.47 90)
+		(unit 1)
+		(exclude_from_sim no)
+		(in_bom yes)
+		(on_board yes)
+		(dnp no)
+		(fields_autoplaced yes)
+		(property "Reference" "R4"
+			(at 71.12 71.12 90)
+			(effects
+				(font
+					(size 1.27 1.27)
+				)
+			)
+		)
+		(property "Value" "2K2"
+			(at 71.12 73.66 90)
+			(effects
+				(font
+					(size 1.27 1.27)
+				)
+			)
+		)
+		(property "Footprint" ""
+			(at 71.12 79.248 90)
+			(effects
+				(font
+					(size 1.27 1.27)
+				)
+				(hide yes)
+			)
+		)
+		(property "Datasheet" "~"
+			(at 71.12 77.47 0)
+			(effects
+				(font
+					(size 1.27 1.27)
+				)
+				(hide yes)
+			)
+		)
+		(property "Description" "Resistor"
+			(at 71.12 77.47 0)
+			(effects
+				(font
+					(size 1.27 1.27)
+				)
+				(hide yes)
+			)
+		)
+		(pin "1"
+		)
+		(pin "2"
+		)
+		(instances
+			(project ""
+				(path "/b82b4682-21bb-43c0-8a97-c0cb83f73104/2638106f-00a2-4c49-9806-0a78e782955a"
+					(reference "R4")
+					(unit 1)
+				)
+			)
+		)
+	)
+	(symbol
 		(lib_id "Transistor_BJT:BC337")
 		(at 83.82 77.47 0)
@@
 	(symbol
 		(lib_id "Device:R_Photo")
-		(at 67.31 85.09 0)
+		(at 59.69 85.09 0)
 		(unit 1)
 		(exclude_from_sim no)
@@
 		(fields_autoplaced yes)
 		(property "Reference" "R3"
-			(at 69.85 83.8199 0)
-			(effects
-				(font
-					(size 1.27 1.27)
-				)
-				(justify left)
-			)
-		)
-		(property "Value" "R_Photo"
-			(at 69.85 86.3599 0)
+			(at 62.23 83.8199 0)
+			(effects
+				(font
+					(size 1.27 1.27)
+				)
+				(justify left)
+			)
+		)
+		(property "Value" "1M"
+			(at 62.23 86.3599 0)
 			(effects
 				(font
@@
 		)
 		(property "Footprint" ""
-			(at 68.58 91.44 90)
+			(at 60.96 91.44 90)
 			(effects
 				(font
@@
 		)
 		(property "Datasheet" "~"
-			(at 67.31 86.36 0)
+			(at 59.69 86.36 0)
 			(effects
 				(font
@@
 		)
 		(property "Description" "Photoresistor"
-			(at 67.31 85.09 0)
+			(at 59.69 85.09 0)
 			(effects
 				(font
@@
 	(symbol
 		(lib_id "power:+3.3V")
-		(at 67.31 54.61 0)
+		(at 59.69 54.61 0)
 		(unit 1)
 		(exclude_from_sim no)
@@
 		(fields_autoplaced yes)
 		(property "Reference" "#PWR04"
-			(at 67.31 58.42 0)
+			(at 59.69 58.42 0)
 			(effects
 				(font
@@
 		)
 		(property "Value" "+3.3V"
-			(at 67.31 49.53 0)
+			(at 59.69 49.53 0)
 			(effects
 				(font
@@
 		)
 		(property "Footprint" ""
-			(at 67.31 54.61 0)
+			(at 59.69 54.61 0)
 			(effects
 				(font
@@
 		)
 		(property "Datasheet" ""
-			(at 67.31 54.61 0)
+			(at 59.69 54.61 0)
 			(effects
 				(font
@@
 		)
 		(property "Description" "Power symbol creates a global label with name \"+3.3V\""
-			(at 67.31 54.61 0)
+			(at 59.69 54.61 0)
 			(effects
 				(font
@@
 	(symbol
 		(lib_id "power:GND")
-		(at 67.31 92.71 0)
+		(at 59.69 92.71 0)
 		(unit 1)
 		(exclude_from_sim no)
@@
 		(fields_autoplaced yes)
 		(property "Reference" "#PWR05"
-			(at 67.31 99.06 0)
+			(at 59.69 99.06 0)
 			(effects
 				(font
@@
 		)
 		(property "Value" "GND"
-			(at 67.31 97.79 0)
+			(at 59.69 97.79 0)
 			(effects
 				(font
@@
 		)
 		(property "Footprint" ""
-			(at 67.31 92.71 0)
+			(at 59.69 92.71 0)
 			(effects
 				(font
@@
 		)
 		(property "Datasheet" ""
-			(at 67.31 92.71 0)
+			(at 59.69 92.71 0)
 			(effects
 				(font
@@
 		)
 		(property "Description" "Power symbol creates a global label with name \"GND\" , ground"
-			(at 67.31 92.71 0)
-			(effects
-				(font
+			(at 59.69 92.71 0)
+			(effects
+				(font

Commit message: fix home work 04
Parts:
- R4: value 2K2 -> 390
Other:
- note added: "V_{control} = 3.3V V_{load} = 12V I_{C_{max}} = 800 - 25% = 600mA hfe = 85 I_{B} = I_{C_{max}} / hfe = 600 / 85 = 7 mA V_{BE} = 0.7V R_{B} = (V_{control} - V_{BE}) / I_{B} = (3.3 - 0.7) / 0.007 = 371,4 Om -> 390"
- note removed: "V_{control} = 3.3V V_{load} = 12V I_{C} = 250mA hfe = 220 I_{B} = I_{C} / hfe = 250 / 220 = 1.14 mA V_{BE} = 0.85V R_{B} = (V_{control} - V_{BE}) / I_{B} = (3.3 - 0.85) / 0.00114 = 2150 Om - 2K2"
Changed lines of the file:
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@@
 		)
 	)
-	(text "V_{control} = 3.3V\nV_{load} = 12V\nI_{C} = 250mA\nhfe = 220\nI_{B} = I_{C} / hfe = 250 / 220 =  1.14 mA\nV_{BE} = 0.85V\nR_{B} = (V_{control} - V_{BE}) / I_{B} = (3.3 - 0.85) / 0.00114 = 2150 Om - 2K2\n"
+	(text "V_{control} = 3.3V\nV_{load} = 12V\n\nI_{C_{max}} = 800 - 25% = 600mA\nhfe = 85\nI_{B} = I_{C_{max}} / hfe = 600 / 85 =  7 mA\nV_{BE} = 0.7V\nR_{B} = (V_{control} - V_{BE}) / I_{B} = (3.3 - 0.7) / 0.007 = 371,4 Om -> 390\n"
 		(exclude_from_sim no)
 		(at 114.554 51.308 0)
@@
 			)
 		)
-		(property "Value" "2K2"
+		(property "Value" "390"
 			(at 71.12 73.66 90)
 			(effects
@@
 		)
 	)
+	(sheet_instances
+		(path "/"
+			(page "1")
+		)
+	)
